Commit message: challenge1.launch launhces puzzlebot model in rviz

File: src/challenge1/puzzlebot_rviz_ch1/urdf/parameters.xacro (robot description, xacro)
@@ -19,6 +19,6 @@
 <xacro:property name="cameraY" value="0.04"/>
 <xacro:property name="cameraZ" value="0.06"/>
-<xacro:property name="mesh_chassis"  value="$(find puzzlebot_rviz)/meshes/chassis.stl" />
-<xacro:property name="mesh_wheel"  value="$(find puzzlebot_rviz)/meshes/wheel.stl" />
-<xacro:property name="mesh_camera"  value="$(find puzzlebot_rviz)/meshes/camera.stl" />
+<xacro:property name="mesh_chassis"  value="$(find puzzlebot_rviz_ch1)/stl_files/MCR2_1000_0_Puzzlebot.stl" />
+<!-- <xacro:property name="mesh_wheel"  value="$(find puzzlebot_rviz_ch1)/meshes/wheel.stl" />
+<xacro:property name="mesh_camera"  value="$(find puzzlebot_rviz_ch1)/meshes/camera.stl" /> -->
 </robot>

File: src/challenge1/puzzlebot_rviz_ch1/urdf/puzzlebot.xacro (robot description, xacro)
@@ -3,8 +3,8 @@
 <robot name="puzzlebot" xmlns:xacro="http://www.ros.org/wiki/xacro">
 <!-- files for gazebo costumization -->
-<xacro:include filename="$(find puzzlebot_rviz)/urdf/parameters.xacro" />
-<xacro:include filename="$(find puzzlebot_rviz)/urdf/macros.xacro" />
-<xacro:include filename="$(find puzzlebot_rviz)/urdf/puzzlebot.gazebo" />
-<xacro:include filename="$(find puzzlebot_rviz)/urdf/materials.xacro" />
+<xacro:include filename="$(find puzzlebot_rviz_ch1)/urdf/parameters.xacro" />
+<xacro:include filename="$(find puzzlebot_rviz_ch1)/urdf/macros.xacro" />
+<xacro:include filename="$(find puzzlebot_rviz_ch1)/urdf/puzzlebot.gazebo" />
+<xacro:include filename="$(find puzzlebot_rviz_ch1)/urdf/materials.xacro" />
 <!-- Dummy link needed to load the model properly-->
   <link name="base_link">
@@ -14,5 +14,6 @@
     <pose>0 0 0 0 0 0</pose>
     <visual>
-      <origin xyz="0 0 0" rpy="${PI/2} 0 ${PI/2}"/>
+      <origin xyz="0 0 0" rpy="0 0 0"/>
+      <!-- <origin xyz="0 0 0" rpy="${PI/2} 0 ${PI/2}"/>         -->
           <geometry>
           	  <mesh filename="file://${mesh_chassis}"/>
